File: HW6.X/ME433/ME433.brd (EAGLE design)
At the start: 100 x 80 mm, 26 parts, among them J1 B, J2 A, U1 PIC32MX170F256B

Commit message: HW6
Parts:
- added J10, J11, J12, J13, J14, J15, J16, J3, J4, J5, J6, J7, J8, J9: (no value), ME433:1X08
- moved J1 261.1 mm to (44.5, 86.4), turned to 90 degrees
- moved J2 257.4 mm to (44.5, 78.7), turned to 90 degrees
- moved R6 251.2 mm to (68.6, 76.2)
- moved U$10 249.6 mm to (54.6, 83.8)
- moved U$9 238.7 mm to (67.3, 69.8)
- moved LED2 191.6 mm to (85.1, 17.8), turned to 90 degrees
- moved R5 190.1 mm to (76.2, 17.8)
- moved R4 189.8 mm to (68.6, 31.8), turned to 270 degrees
- moved C4 184.7 mm to (73.7, 34.3), turned to 90 degrees
- moved R3 183.5 mm to (64.8, 31.8), turned to 270 degrees
- moved U$8 179.3 mm to (82.5, 41.9), turned to 270 degrees
- moved C1 130.7 mm to (57.1, 57.1), turned to 90 degrees
- moved R2 125.7 mm to (29.2, 68.6), turned to 270 degrees
- moved U$5 123.3 mm to (35.6, 71.1)
- moved C3 121.1 mm to (55.9, 34.3), turned to 270 degrees
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Connections:
- new net N$10: J3.8, J4.8, J5.8, J6.8, J7.8
- new net N$11: J3.7, J4.7, J5.7, J6.7, J7.7
- new net N$12: J3.6, J4.6, J5.6, J6.6, J7.6
- new net N$13: J3.5, J4.5, J5.5, J6.5, J7.5
- new net N$14: J3.4, J4.4, J5.4, J6.4, J7.4
- new net N$15: J3.3, J4.3, J5.3, J6.3, J7.3
- new net N$16: J3.2, J4.2, J5.2, J6.2, J7.2
- new net N$17: J3.1, J4.1, J5.1, J6.1, J7.1
- new net N$18: J10.8, J11.8, J12.8, J8.8, J9.8
- new net N$19: J10.7, J11.7, J12.7, J8.7, J9.7
- new net N$20: J10.6, J11.6, J12.6, J8.6, J9.6
- new net N$21: J10.5, J11.5, J12.5, J8.5, J9.5
- new net N$22: J10.4, J11.4, J12.4, J8.4, J9.4
- new net N$23: J10.3, J11.3, J12.3, J8.3, J9.3
- new net N$24: J10.2, J11.2, J12.2, J8.2, J9.2
- new net N$25: J10.1, J11.1, J12.1, J8.1, J9.1
- net +3V3: now also J13.1, J13.2, J13.3, J13.4, J13.5, J13.6, J13.7, J13.8, J16.1, J16.2, J16.3, J16.4, J16.5, J16.6, J16.7, J16.8, R6.2
- net GND: now also J14.1, J14.2, J14.3, J14.4, J14.5, J14.6, J14.7, J14.8, J15.1, J15.2, J15.3, J15.4, J15.5, J15.6, J15.7, J15.8
Routing:
- net +3V3: track 0.00 -> 319.8 mm, vias 0 -> 6
- net VIN: track 0.00 -> 72.2 mm
- net B15: track 0.00 -> 62.3 mm, vias 0 -> 2
- net B13: track 0.00 -> 58.7 mm
- net BPWM: track 0.00 -> 58.3 mm
- net BDIR: track 0.00 -> 57.2 mm, vias 0 -> 2
- net APWM: track 0.00 -> 54.0 mm
- net B12: track 0.00 -> 53.8 mm
- net ADIR: track 0.00 -> 53.3 mm
- net B14: track 0.00 -> 52.7 mm
- net B9: track 0.00 -> 41.6 mm
- net B8: track 0.00 -> 38.4 mm, vias 0 -> 2
- net N$26: track 0.00 -> 30.8 mm
- net N$6: track 0.00 -> 28.6 mm
- net MCLR: track 0.00 -> 25.6 mm
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- added copper zone on layer 16, net GND
Other:
- board size 100 x 80 mm -> 100 x 100 mm
- board text added: "3.3V"
- board text added: "A"
- board text added: "B"
- board text added: "Bohan Yao"
- board text added: "GND"
- board text added: "ME433"
