File: HW6.X/ME433/ME433.sch (EAGLE design)
At the start: 1 part, among them U1 PIC32MX170F256B

Commit message: HW6 (partial) + 8
Parts:
- added BAT: (no value), ME433:CONN_02
- added C1, C4: 0.1uF, ME433:C-US025-030X050
- added C2: 0.1 uF, ME433:C-US025-030X050
- added C3: 10uF, ME433:CPOL-USB45181A
- added J1: B, ME433:CONN_02
- added J2: A, ME433:CONN_02
- added LED1: RED, ME433:LED3MM
- added LED2: GREEN, ME433:LED3MM
- added R1, R5: 330, ME433:R-US_0207/10
- added R2, R3, R4, R6: 10k, ME433:R-US_0207/10
- added U$1: MICROUSB, ME433:MICROUSB
- added U$10: HBRIDGE, ME433:HBRIDGE
- added U$2: SLIDE, ME433:SLIDE
- added U$3: POLOLU3V3, ME433:POLOLU3V3
- added U$4: SNAP, ME433:SNAP
- added U$5: RESET, ME433:PUSH
- added U$6: UART-USB, ME433:UART-USB
- added U$7: LCD, ME433:LCD
- added U$8: IOEXPANDER, ME433:IOEXPANDER
- added U$9: USER, ME433:PUSH
Connections:
- new net +3V3: C1.1, C2.1, C4.1, LED1.A, R2.2, R3.2, R4.2, U$10.13.VCC, U$10.8.MD, U$3.1.VOUT, U$4.2.VDD, U$7.2.VCC, U$8.18.RESET, U$8.9.VDD, U1.13.VDD, U1.28.AVDD
- new net +5V: U$1.1.VBUS, U$2.1.VBUS
- new net ADIR: U$10.9.IN1-PH-A, U$8.22.A1
- new net APWM: U$10.10.IN2-EN-A, U$8.23.A2
- new net B0-PGD: U$4.4.PGD, U1.4.B0-PGD
- new net B1-PGC: U$4.5.PGC, U1.5.B1-PGC
- new net B12: U$7.6.DC, U1.23.B12
- new net B13: U$6.5.RXD, U$7.4.SDA, U1.24.B13
- new net B14: U$7.3.SCL, U1.25.B14
- new net B15: U$6.4.TXD, U$7.5.RESET, U1.26.B15
- new net B8: R3.1, U$8.12.SCK, U1.17.B8
- new net B9: R4.1, U$8.13.SDA, U1.18.B9
- new net BDIR: U$10.11.IN1-PH-B, U$8.24.A3
- new net BPWM: U$10.12.IN2-EN-B, U$8.25.A4
- new net GND: BAT.1, C1.2, C2.2, C3.-, C4.2, R1.1, R5.1, U$1.5.GND, U$10.1.GND, U$10.14.GND, U$3.2.GND, U$4.3.GND, U$5.2, U$6.1.GND, U$7.1.GND, U$8.10.VSS, U$8.15.A0, U$8.16.A1, U$8.17.A2, U1.19.VSS, U1.27.AVSS, U1.8.VSS
- new net MCLR: R2.1, U$4.1.MCLR, U$5.1, U1.1.MCLR
- new net N$1: LED1.C, R1.2
- new net N$2: J1.2, U$10.3.O2B
- new net N$3: C3.+, U1.20.VCAP
- new net N$4: J1.1, U$10.4.O1B
- new net N$5: R6.1, U$8.1.B0, U$9.1
- new net N$6: LED2.A, U$8.21.A0
- new net N$7: LED2.C, R5.2
- new net N$8: J2.2, U$10.5.O2A
- new net N$9: J2.1, U$10.6.O1A
- new net V+: BAT.2, U$2.3.VBAT
- new net VIN: U$10.2.VIN, U$2.2.VOUT, U$3.3.VIN
Other:
- note added: "B12 - DC"
- note added: "B13 - U1RX, SDO1"
- note added: "B14 - SCK1"
- note added: "B15 - U1TX, RES"
- note added: "B8 - SCL1"
- note added: "B9 - SDA1"
- moved on the sheet: U1

Commit message: HW6
Parts:
- added J10, J11, J12, J13, J14, J15, J16, J3, J4, J5, J6, J7, J8, J9: (no value), ME433:CONN_08"
Connections:
- new net N$10: J3.8, J4.8, J5.8, J6.8, J7.8
- new net N$11: J3.7, J4.7, J5.7, J6.7, J7.7
- new net N$12: J3.6, J4.6, J5.6, J6.6, J7.6
- new net N$13: J3.5, J4.5, J5.5, J6.5, J7.5
- new net N$14: J3.4, J4.4, J5.4, J6.4, J7.4
- new net N$15: J3.3, J4.3, J5.3, J6.3, J7.3
- new net N$16: J3.2, J4.2, J5.2, J6.2, J7.2
- new net N$17: J3.1, J4.1, J5.1, J6.1, J7.1
- new net N$18: J10.8, J11.8, J12.8, J8.8, J9.8
- new net N$19: J10.7, J11.7, J12.7, J8.7, J9.7
- new net N$20: J10.6, J11.6, J12.6, J8.6, J9.6
- new net N$21: J10.5, J11.5, J12.5, J8.5, J9.5
- new net N$22: J10.4, J11.4, J12.4, J8.4, J9.4
- new net N$23: J10.3, J11.3, J12.3, J8.3, J9.3
- new net N$24: J10.2, J11.2, J12.2, J8.2, J9.2
- new net N$25: J10.1, J11.1, J12.1, J8.1, J9.1
- net +3V3: now also J13.1, J13.2, J13.3, J13.4, J13.5, J13.6, J13.7, J13.8, J16.1, J16.2, J16.3, J16.4, J16.5, J16.6, J16.7, J16.8, R6.2
- net GND: now also J14.1, J14.2, J14.3, J14.4, J14.5, J14.6, J14.7, J14.8, J15.1, J15.2, J15.3, J15.4, J15.5, J15.6, J15.7, J15.8
